File: KicadSchematics/newkicad/ScoreBoxLite/ScoreBoxLite.kicad_sch (KiCad schematic)
At the start: 59 parts, among them J3 Screw_Terminal_01x05, J4 Screw_Terminal_01x02, Q1 AO3400A, U1 ESP32-WROOM-32E, U2 SN74AHCT125N

Commit message: added part buttons
Connections:
- net MatrixIO: now also U1.11 (IO26)
- net SpeakerIO: now also U1.12 (IO27)
- net ReArmButton: now reaches U1.13 (IO14)
- net VolumeButton: now reaches U1.16 (IO13)
- net ModeButton: now reaches U1.27 (IO16)
- net PowerButton: now reaches U1.28 (IO17)
Changed lines of the file:
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@@
+	(wire
+		(pts
+			(xy 205.74 204.47) (xy 209.55 204.47)
+		)
+		(stroke
+			(width 0)
+			(type default)
+		)
+	)
 	(wire
 		(pts
@@
 	(wire
 		(pts
+			(xy 205.74 201.93) (xy 209.55 201.93)
+		)
+		(stroke
+			(width 0)
+			(type default)
+		)
+	)
+	(wire
+		(pts
 			(xy 365.76 151.13) (xy 365.76 153.67)
 		)
@@
 	(wire
 		(pts
+			(xy 205.74 176.53) (xy 209.55 176.53)
+		)
+		(stroke
+			(width 0)
+			(type default)
+		)
+	)
+	(wire
+		(pts
 			(xy 210.82 95.25) (xy 220.98 95.25)
 		)
@@
 	(wire
 		(pts
+			(xy 205.74 181.61) (xy 209.55 181.61)
+		)
+		(stroke
+			(width 0)
+			(type default)
+		)
+	)
+	(wire
+		(pts
 			(xy 283.21 64.77) (xy 283.21 74.93)
 		)
@@
 	(wire
 		(pts
+			(xy 205.74 184.15) (xy 209.55 184.15)
+		)
+		(stroke
+			(width 0)
+			(type default)
+		)
+	)
+	(wire
+		(pts
 			(xy 384.81 106.68) (xy 391.16 106.68)
 		)
@@
 		(pts
 			(xy 265.43 106.68) (xy 265.43 105.41)
+		)
+		(stroke
+			(width 0)
+			(type default)
+		)
+	)
+	(wire
+		(pts
+			(xy 205.74 173.99) (xy 209.55 173.99)
 		)
 		(stroke
@@
 		)
 	)
+	(label "PowerButton"
+		(at 337.82 187.96 180)
+		(effects
+			(font
+				(size 1.27 1.27)
+			)
+			(justify right bottom)
+		)
+	)
 	(label "RedCloseIO"
 		(at 167.64 163.83 180)
@@
 		)
 	)
+	(label "SpeakerIO"
+		(at 209.55 204.47 0)
+		(effects
+			(font
+				(size 1.27 1.27)
+			)
+			(justify left bottom)
+		)
+	)
 	(label "GreenGNDInput"
 		(at 210.82 95.25 0)
@@
 		)
 	)
+	(label "ReArmButton"
+		(at 209.55 176.53 0)
+		(effects
+			(font
+				(size 1.27 1.27)
+			)
+			(justify left bottom)
+		)
+	)
 	(label "RedMidInput"
 		(at 99.06 64.77 0)
@@
 		)
 	)
+	(label "VolumeButton"
+		(at 337.82 198.12 180)
+		(effects
+			(font
+				(size 1.27 1.27)
+			)
+			(justify right bottom)
+		)
+	)
 	(label "MatrixIO"
 		(at 350.52 110.49 180)
@@
 		)
 	)
+	(label "PowerButton"
+		(at 209.55 184.15 0)
+		(effects
+			(font
+				(size 1.27 1.27)
+			)
+			(justify left bottom)
+		)
+	)
 	(label "RedCloseIO"
 		(at 176.53 30.48 0)
@@
 		)
 	)
+	(label "VolumeButton"
+		(at 209.55 173.99 0)
+		(effects
+			(font
+				(size 1.27 1.27)
+			)
+			(justify left bottom)
+		)
+	)
 	(label "GreenCloseInput"
 		(at 210.82 30.48 0)
@@
 		)
 	)
+	(label "MatrixIO"
+		(at 209.55 201.93 0)
+		(effects
+			(font
+				(size 1.27 1.27)
+			)
+			(justify left bottom)
+		)
+	)
+	(label "ReArmButton"
+		(at 337.82 195.58 180)
+		(effects
+			(font
+				(size 1.27 1.27)
+			)
+			(justify right bottom)
+		)
+	)
 	(label "RedMidIO"
 		(at 176.53 64.77 0)
@@
 		(effects
 			(font
+				(size 1.27 1.27)
+			)
+			(justify left bottom)
+		)
+	)
+	(label "ModeButton"
+		(at 337.82 190.5 180)
+		(effects
+			(font
+				(size 1.27 1.27)
+			)
+			(justify right bottom)
+		)
+	)
+	(label "ModeButton"
+		(at 209.55 181.61 0)
+		(effects
+			(font
