File: KicadSchematics/newkicad/ScoreBoxLite/ScoreBoxLite.kicad_sch (KiCad schematic)
At the start: 59 parts, among them J3 Screw_Terminal_01x05, J4 Screw_Terminal_01x02, Q1 AO3400A, U1 ESP32-WROOM-32E, U2 SN74AHCT125N

Commit message: adding idek what now
Connections:
- net GreenCloseIO: now also U1.6 (IO34); no longer U1.7 (IO35)
- net MatrixIO: now also U1.11 (IO26)
- net RedGNDIO: now also U1.7 (IO35); no longer U1.6 (IO34)
Changed lines of the file:
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@@
+	(wire
+		(pts
+			(xy 205.74 201.93) (xy 209.55 201.93)
+		)
+		(stroke
+			(width 0)
+			(type default)
+		)
+	)
 	(wire
 		(pts
@@
 		)
 	)
+	(label "MatrixIO"
+		(at 209.55 201.93 0)
+		(effects
+			(font
+				(size 1.27 1.27)
+			)
+			(justify left bottom)
+		)
+	)
 	(label "RedMidIO"
 		(at 176.53 64.77 0)
@@
 		)
 	)
-	(label "GreenCloseIO"
+	(label "RedGNDIO"
 		(at 209.55 214.63 0)
 		(effects
@@
 		)
 	)
-	(label "RedGNDIO"
+	(label "GreenCloseIO"
 		(at 209.55 212.09 0)
 		(effects
